File: orphkicad.kicad_pcb (KiCad board)
At the start: 2 copper layers, 21 x 51 mm, 41 parts, among them J1 USB_C_Receptacle_USB2.0_16P, J2 SWD, SW1 BTN_BOOT, SW2 BTN_RST, SW3 BTN_USR, U1 RP2040, U2 W25Q16JVUXIQ, U3 USBLC6-2SC6, U5 XC6206PxxxMR, X1 X322512MOB4SI 12pF

Commit message: minor fixes + stitching vias
Routing:
- net GND: track 22.8 -> 17.6 mm, vias 50 -> 64
