File: orphkicad.kicad_sch (KiCad schematic)
At the start: 41 parts, among them J1 USB_C_Receptacle_USB2.0_16P, J2 SWD, SW1 BTN_BOOT, SW2 BTN_RST, SW3 BTN_USR, U1 RP2040, U2 W25Q16JVUXIQ, U3 USBLC6-2SC6, U5 XC6206PxxxMR, X1 X322512MOB4SI 12pF

Commit message: updated dnp
Parts:
- H1, H2, J2, JP1: now not fitted
- R5, R6: now fitted
Changed lines of the file:
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@@
 		(in_bom yes)
 		(on_board yes)
-		(dnp yes)
+		(dnp no)
 		(property "Reference" "R6"
 			(at 136.525 95.885 90)
@@
 		(in_bom yes)
 		(on_board yes)
-		(dnp no)
+		(dnp yes)
 		(property "Reference" "JP1"
 			(at 231.775 68.58 0)
@@
 		(in_bom yes)
 		(on_board yes)
-		(dnp yes)
+		(dnp no)
 		(property "Reference" "R5"
 			(at 136.525 89.535 90)
@@
 		(in_bom yes)
 		(on_board yes)
-		(dnp no)
+		(dnp yes)
 		(fields_autoplaced yes)
 		(property "Reference" "J2"
@@
 		(in_bom yes)
 		(on_board yes)
-		(dnp no)
+		(dnp yes)
 		(property "Reference" "H1"
 			(at 30.48 144.78 0)
@@
 		(in_bom yes)
 		(on_board yes)
-		(dnp no)
+		(dnp yes)
 		(property "Reference" "H2"
 			(at 47.625 144.78 0)
