File: orphkicad.kicad_sch (KiCad schematic)
At the start: 41 parts, among them J1 USB_C_Receptacle_USB2.0_16P, J2 SWD, SW1 BTN_BOOT, SW2 BTN_RST, SW3 BTN_USR, U1 RP2040, U2 W25Q16JVUXIQ, U3 USBLC6-2SC6, U5 XC6206PxxxMR, X1 X322512MOB4SI 12pF

Commit message: Remove extra space from LCSC Part #
Parts:
- J1: LCSC C2765186 -> C2765186
- SW1, SW2, SW3: LCSC C455280 -> C455280
Changed lines of the file:
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@@
 			)
 		)
-		(property "LCSC" "C455280 "
+		(property "LCSC" "C455280"
 			(at 91.44 196.215 0)
 			(effects
@@
 			)
 		)
-		(property "LCSC" "C2765186 "
+		(property "LCSC" "C2765186"
 			(at 119.38 101.6 0)
 			(effects
@@
 			)
 		)
-		(property "LCSC" "C455280 "
+		(property "LCSC" "C455280"
 			(at 163.83 47.625 0)
 			(effects
@@
 			)
 		)
-		(property "LCSC" "C455280 "
+		(property "LCSC" "C455280"
 			(at 91.44 185.42 0)
 			(effects
