File: testboard/testboard/testboard.kicad_pcb (KiCad board)
At the start: 2 copper layers, 65 x 55 mm, 62 parts

Commit message: FIXIEMIDNWJKE
Parts:
- R32: footprint Package_TO_SOT_SMD:TO-263-2_TabPin1 -> Package_TO_SOT_SMD:TO-263-2
Connections:
- R32 pad 2: +5V -> unconnected-(R32-Pad2)
Routing:
- net GND: track 12.9 -> 8.13 mm, vias 46 -> 5
- net unconnected-(R32-Pad2): vias 0 -> 44
- added copper zone on B.Cu, net unconnected-(R32-Pad2)
- added copper zone on F.Cu, net unconnected-(R32-Pad2)
- removed copper zone on F.Cu, net GND
