File: testboard/testboard/testboard.kicad_sch (KiCad schematic)
At the start: 62 parts

Commit message: FIXIEMIDNWJKE
Parts:
- R32: footprint Package_TO_SOT_SMD:TO-263-2_TabPin1 -> Package_TO_SOT_SMD:TO-263-2; symbol Device:R -> Device:R_Potentiometer
Connections:
- net +5V: now also R32.3; no longer R32.2
Changed lines of the file:
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@@
 	)
 	(symbol
-		(lib_id "Device:R")
+		(lib_id "Device:R_Potentiometer")
 		(at 168.91 125.73 180)
 		(unit 1)
@@
 			)
 		)
-		(property "Footprint" "Package_TO_SOT_SMD:TO-263-2_TabPin1"
-			(at 170.688 125.73 90)
+		(property "Footprint" "Package_TO_SOT_SMD:TO-263-2"
+			(at 168.91 125.73 0)
 			(effects
 				(font
@@
 			)
 		)
-		(property "Description" "Resistor"
+		(property "Description" "Potentiometer"
 			(at 168.91 125.73 0)
 			(effects
@@
 		(pin "2"
 		)
+		(pin "3"
+		)
 		(instances
